Commit message: New TWIP; using proper pitch for reward

File: assets/urdf/twip/twip.urdf (robot description, URDF)
Before this commit: robot twip, 4 links, 3 joints
Links:
- removed link centre
- link body: mass 2.0 -> 1.1781; geometry collision mesh filename=meshes/body_collision.stl; visual mesh filename=meshes/body_visual.stl
- link left_wheel: mass 0.3 -> 0.410645; geometry collision mesh filename=meshes/left_wheel_collision.stl; visual mesh filename=meshes/left_wheel_visual.stl
- link right_wheel: mass 0.3 -> 0.410645; geometry collision mesh filename=meshes/right_wheel_collision.stl; visual mesh filename=meshes/right_wheel_visual.stl
Joints:
- removed joint centre_frame
- joint lwheel: limit effort=1 -> effort=1 velocity=20; origin xyz=-0.155 0 -0.41 rpy=1.5708 -0 1.5708 -> xyz=-0.135148 -2.90755e-05 -0.03878 rpy=1.5708 -0 1.5708
- joint rwheel: limit effort=1 -> effort=1 velocity=20; origin xyz=0.155 0 -0.41 rpy=-1.5708 -0 1.5708 -> xyz=0.135148 2.90755e-05 -0.03878 rpy=-1.5708 -0 1.5708

Commit message: new twip design 2.0

File: assets/urdf/twip/twip.urdf (robot description, URDF)
Before this commit: robot twip, 3 links, 2 joints
Links:
- link body: mass 1.1781 -> 0.850962
Joints:
- joint lwheel: origin xyz=-0.135148 -2.90755e-05 -0.03878 rpy=1.5708 -0 1.5708 -> xyz=0.0509238 -0.0784359 -0.0289244 rpy=-3.14159 1.5708 0
- joint rwheel: axis 0 0 1 -> 0 0 -1; origin xyz=0.135148 2.90755e-05 -0.03878 rpy=-1.5708 -0 1.5708 -> xyz=-0.219373 -0.078494 -0.0289244 rpy=1.66533e-16 1.5708 0

Commit message: fixed masses

File: assets/urdf/twip/twip.urdf (robot description, URDF)
Before this commit: robot twip, 3 links, 2 joints
Links:
- link body: mass 0.850962 -> 2.02723
- link left_wheel: mass 0.410645 -> 0.190998
- link right_wheel: mass 0.410645 -> 0.190998

Commit message: fixed battery mass

File: assets/urdf/twip/twip.urdf (robot description, URDF)
Before this commit: robot twip, 3 links, 2 joints
Links:
- link body: mass 2.02723 -> 2.24123
